File: hardware/Rev 1.0/hfm_adapter_nucleo-32.sch (EAGLE design)
At the start: 50 parts, among them IC1 NUCLEO-G431KB, IC10 OPA2992D, IC11 OPA2172D, IC2 M24M02, IC3 IP4234CZ6,115, IC4 LPS25HBTR, IC5 REF02D, IC6 SRV05-4MR6T1GTSSOP6, IC8 TLE42764_ADJDV, IC9 TLE4252D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

Commit message: some values changed, BOM added
Parts:
- R10, R7: value 10k 0.5% -> 17k 0.5%
- R11, R8: value 5k1 0.5% -> 33k 0.5%
- R3, R5: value 18k 0.5% -> 17k 0.5%
Other:
- note added: "VIN is 10v, because of 5v output of OpAmps. OpAmps are running with gain of 1.515"
- note added: "Voltage divider faktor: 33k / (17k +33k) = 0.66"
- note removed: "VIN is 10v, because of 5v output of OpAmps. OpAmps are running with gain of 1.510"
- note removed: "Voltage divider faktor: 18k / 33k = 0.64705882"
Changed lines of the file:
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@@
 <part name="U$12" library="microbuilder" deviceset="GND" device=""/>
 <part name="U$16" library="microbuilder" deviceset="GND" device=""/>
-<part name="R3" library="rcl" library_urn="urn:adsk.eagle:library:334" deviceset="R-EU_" device="R0805" package3d_urn="urn:adsk.eagle:package:23553/2" value="18k 0.5%"/>
+<part name="R3" library="rcl" library_urn="urn:adsk.eagle:library:334" deviceset="R-EU_" device="R0805" package3d_urn="urn:adsk.eagle:package:23553/2" value="17k 0.5%"/>
 <part name="R4" library="rcl" library_urn="urn:adsk.eagle:library:334" deviceset="R-EU_" device="R0805" package3d_urn="urn:adsk.eagle:package:23553/2" value="33k 0.5%"/>
 <part name="C4" library="rcl" library_urn="urn:adsk.eagle:library:334" deviceset="C-EU" device="C0805" package3d_urn="urn:adsk.eagle:package:23617/2" value="100nF"/>
@@
 <part name="U$37" library="microbuilder" deviceset="3.3V" device=""/>
 <part name="U$39" library="microbuilder" deviceset="GND" device=""/>
-<part name="R7" library="rcl" library_urn="urn:adsk.eagle:library:334" deviceset="R-EU_" device="R0805" package3d_urn="urn:adsk.eagle:package:23553/2" value="10k 0.5%"/>
-<part name="R8" library="rcl" library_urn="urn:adsk.eagle:library:334" deviceset="R-EU_" device="R0805" package3d_urn="urn:adsk.eagle:package:23553/2" value="5k1 0.5%"/>
-<part name="R10" library="rcl" library_urn="urn:adsk.eagle:library:334" deviceset="R-EU_" device="R0805" package3d_urn="urn:adsk.eagle:package:23553/2" value="10k 0.5%"/>
-<part name="R11" library="rcl" library_urn="urn:adsk.eagle:library:334" deviceset="R-EU_" device="R0805" package3d_urn="urn:adsk.eagle:package:23553/2" value="5k1 0.5%"/>
+<part name="R7" library="rcl" library_urn="urn:adsk.eagle:library:334" deviceset="R-EU_" device="R0805" package3d_urn="urn:adsk.eagle:package:23553/2" value="17k 0.5%"/>
+<part name="R8" library="rcl" library_urn="urn:adsk.eagle:library:334" deviceset="R-EU_" device="R0805" package3d_urn="urn:adsk.eagle:package:23553/2" value="33k 0.5%"/>
+<part name="R10" library="rcl" library_urn="urn:adsk.eagle:library:334" deviceset="R-EU_" device="R0805" package3d_urn="urn:adsk.eagle:package:23553/2" value="17k 0.5%"/>
+<part name="R11" library="rcl" library_urn="urn:adsk.eagle:library:334" deviceset="R-EU_" device="R0805" package3d_urn="urn:adsk.eagle:package:23553/2" value="33k 0.5%"/>
 <part name="U$43" library="microbuilder" deviceset="GND" device=""/>
 <part name="U$44" library="microbuilder" deviceset="GND" device=""/>
@@
 <part name="IC6" library="Heinrich" deviceset="SRV05-4MR6T1G" device="TSSOP6"/>
 <part name="U$18" library="microbuilder" deviceset="GND" device=""/>
-<part name="R5" library="rcl" library_urn="urn:adsk.eagle:library:334" deviceset="R-EU_" device="R0805" package3d_urn="urn:adsk.eagle:package:23553/2" value="18k 0.5%"/>
+<part name="R5" library="rcl" library_urn="urn:adsk.eagle:library:334" deviceset="R-EU_" device="R0805" package3d_urn="urn:adsk.eagle:package:23553/2" value="17k 0.5%"/>
 <part name="R6" library="rcl" library_urn="urn:adsk.eagle:library:334" deviceset="R-EU_" device="R0805" package3d_urn="urn:adsk.eagle:package:23553/2" value="33k 0.5%"/>
 <part name="R13" library="rcl" library_urn="urn:adsk.eagle:library:334" deviceset="R-EU_" device="R0805" package3d_urn="urn:adsk.eagle:package:23553/2" value="82k"/>
@@
 <plain>
 <text x="121.92" y="160.02" size="1.778" layer="97">Voltage divider faktor:
-18k / 33k = 0.64705882</text>
+33k / (17k +33k) = 0.66</text>
 </plain>
 <instances>
@@
 <plain>
 <text x="93.98" y="157.48" size="1.778" layer="97">VIN is 10v, because of 5v output of OpAmps.
-OpAmps are running with gain of 1.510</text>
+OpAmps are running with gain of 1.515</text>
 </plain>
 <instances>
@@
 <plain>
 <text x="66.04" y="149.86" size="1.778" layer="97">VIN is 10v, because of 5v output of OpAmps.
-OpAmps are running with gain of 1.510</text>
+OpAmps are running with gain of 1.515</text>
 </plain>
 <instances>
