File: hardware/Rev1.1/hfm_adapter_nucleo-32.sch (EAGLE design)
At the start: 50 parts, among them IC1 NUCLEO-G431KB, IC10 OPA2992D, IC11 OPA2172D, IC2 M24M02, IC3 IP4234CZ6,115, IC4 LPS25HBTR, IC6 SRV05-4MR6T1GTSSOP6, IC7 TLE4252D, IC8 TLE42764DV, IC9 ADR01_02_03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

Commit message: some small changes
Other:
- note added: "VIN is 10v, because of 5v output of OpAmps. OpAmps are running with gain of 1.56"
- note removed: "VIN is 10v, because of 5v output of OpAmps. OpAmps are running with gain of 1.515"
Changed lines of the file:
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@@
 <part name="U$13" library="microbuilder" deviceset="5.0V" device=""/>
 <part name="U$51" library="microbuilder" deviceset="5.0V" device=""/>
-<part name="U$53" library="microbuilder" deviceset="GND" device=""/>
 <part name="C11" library="rcl" library_urn="urn:adsk.eagle:library:334" deviceset="C-EU" device="C0805" package3d_urn="urn:adsk.eagle:package:23617/2" value="1uF"/>
 <part name="U$54" library="microbuilder" deviceset="GND" device=""/>
@@
 <plain>
 <text x="66.04" y="149.86" size="1.778" layer="97">VIN is 10v, because of 5v output of OpAmps.
-OpAmps are running with gain of 1.515</text>
+OpAmps are running with gain of 1.56</text>
 </plain>
 <instances>
@@
 <instance part="U$26" gate="G$1" x="114.3" y="127"/>
 <instance part="U$50" gate="G$1" x="132.08" y="142.24" rot="R270"/>
-<instance part="U$53" gate="G$1" x="124.46" y="35.56"/>
 <instance part="C11" gate="G$1" x="124.46" y="137.16"/>
 <instance part="U$54" gate="G$1" x="124.46" y="127"/>
