File: hardware/Rev1.1/hfm_adapter_nucleo-32.brd (EAGLE design)
At the start: 101.6 x 82.5 mm, 50 parts, among them IC1 NUCLEO-G431KB, IC10 OPA2992D, IC11 OPA2172D, IC2 M24M02, IC3 IP4234CZ6,115, IC4 LPS25HBTR, IC6 SRV05-4MR6T1GTSSOP6, IC7 TLE4252D, IC8 TLE42764DV, IC9 ADR01_02_03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

Commit message: amplification factor corrected
Parts:
- R10, R7: value 5k6 0.5% -> 10k 0.5%
- R11, R8: value 10k 0.5% -> 5k6 0.5%
Changed lines of the file:
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@@
 <attribute name="SPICEPREFIX" value="R" x="77.47" y="50.8" size="1.778" layer="27" rot="R180" display="off"/>
 </element>
-<element name="R10" library="rcl" library_urn="urn:adsk.eagle:library:334" package="R0805" package3d_urn="urn:adsk.eagle:package:23553/2" value="5k6 0.5%" x="54.61" y="43.18" smashed="yes">
+<element name="R10" library="rcl" library_urn="urn:adsk.eagle:library:334" package="R0805" package3d_urn="urn:adsk.eagle:package:23553/2" value="10k 0.5%" x="54.61" y="43.18" smashed="yes">
 <attribute name="NAME" x="57.15" y="42.545" size="0.762" layer="25" font="vector"/>
 <attribute name="SPICEPREFIX" value="R" x="54.61" y="43.18" size="1.778" layer="27" display="off"/>
 </element>
-<element name="R11" library="rcl" library_urn="urn:adsk.eagle:library:334" package="R0805" package3d_urn="urn:adsk.eagle:package:23553/2" value="10k 0.5%" x="54.61" y="40.64" smashed="yes" rot="R180">
+<element name="R11" library="rcl" library_urn="urn:adsk.eagle:library:334" package="R0805" package3d_urn="urn:adsk.eagle:package:23553/2" value="5k6 0.5%" x="54.61" y="40.64" smashed="yes" rot="R180">
 <attribute name="NAME" x="57.15" y="40.005" size="0.762" layer="25" font="vector"/>
 <attribute name="SPICEPREFIX" value="R" x="54.61" y="40.64" size="1.778" layer="27" rot="R180" display="off"/>
@@
 <attribute name="SPICEPREFIX" value="R" x="69.85" y="45.72" size="1.778" layer="27" display="off"/>
 </element>
-<element name="R7" library="rcl" library_urn="urn:adsk.eagle:library:334" package="R0805" package3d_urn="urn:adsk.eagle:package:23553/2" value="5k6 0.5%" x="53.34" y="25.4" smashed="yes">
+<element name="R7" library="rcl" library_urn="urn:adsk.eagle:library:334" package="R0805" package3d_urn="urn:adsk.eagle:package:23553/2" value="10k 0.5%" x="53.34" y="25.4" smashed="yes">
 <attribute name="NAME" x="55.88" y="25.4" size="0.762" layer="25" font="vector"/>
 <attribute name="SPICEPREFIX" value="R" x="53.34" y="25.4" size="1.778" layer="27" display="off"/>
 </element>
-<element name="R8" library="rcl" library_urn="urn:adsk.eagle:library:334" package="R0805" package3d_urn="urn:adsk.eagle:package:23553/2" value="10k 0.5%" x="53.34" y="27.94" smashed="yes" rot="R180">
+<element name="R8" library="rcl" library_urn="urn:adsk.eagle:library:334" package="R0805" package3d_urn="urn:adsk.eagle:package:23553/2" value="5k6 0.5%" x="53.34" y="27.94" smashed="yes" rot="R180">
 <attribute name="NAME" x="55.88" y="27.94" size="0.762" layer="25" font="vector"/>
 <attribute name="SPICEPREFIX" value="R" x="53.34" y="27.94" size="1.778" layer="27" rot="R180" display="off"/>
